File: Filter.kicad_pcb (KiCad board)
At the start: 2 copper layers, 85.3 x 49 mm, 47 parts, among them J1 Conn_Coaxial, J3 Conn_01x04_Pin, J4 Conn_Coaxial, T1 BN-43-2402, T2 BN-43-2402, U1 SN74CBT3253, U2 SN74CBT3253

Commit message: Changes.
Routing:
- net +5V: track 134.6 -> 137.4 mm
Changed lines of the file:
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@@
       (drillshape 0)
       (scaleselection 1)
-      (outputdirectory "Gerber/")
+      (outputdirectory "Gerber/Drill/")
     )
   )
@@
   (segment (start 125.9 70.81) (end 123.6 70.81) (width 2) (layer "B.Cu") (net 2))
   (segment (start 194.07 90.83) (end 194.07 85.75) (width 2) (layer "B.Cu") (net 2))
-  (segment (start 133.8675 102.9025) (end 134.74 102.03) (width 0.4) (layer "F.Cu") (net 3))
   (segment (start 182.865 89.89) (end 183.885 90.91) (width 0.4) (layer "F.Cu") (net 3))
-  (segment (start 133.8675 104.2675) (end 133.8675 102.9025) (width 0.4) (layer "F.Cu") (net 3))
+  (segment (start 181.19 109.47) (end 140.77 109.47) (width 0.4) (layer "F.Cu") (net 3))
   (segment (start 183.885 90.91) (end 184.365 90.91) (width 0.4) (layer "F.Cu") (net 3))
-  (segment (start 154.89 104.57) (end 141.3 104.57) (width 0.4) (layer "F.Cu") (net 3))
+  (segment (start 138.71 107.41) (end 138.71 102.08) (width 0.4) (layer "F.Cu") (net 3))
   (segment (start 138.71125 101.98125) (end 138.71125 96.4925) (width 0.4) (layer "F.Cu") (net 3))
   (segment (start 136.47375 93.77) (end 136.43375 93.81) (width 0.4) (layer "F.Cu") (net 3))
@@
   (segment (start 136.47375 95.1525) (end 136.94125 95.62) (width 0.4) (layer "F.Cu") (net 3))
   (segment (start 183.115 88.12) (end 184.245 88.12) (width 0.4) (layer "F.Cu") (net 3))
-  (segment (start 185.8 93.39) (end 185.8 104.86) (width 0.4) (layer "F.Cu") (net 3))
+  (segment (start 184.365 91.955) (end 185.8 93.39) (width 0.4) (layer "F.Cu") (net 3))
+  (segment (start 138.6625 102.03) (end 134.74 102.03) (width 0.4) (layer "F.Cu") (net 3))
   (segment (start 134.49125 93.81) (end 133.83125 94.47) (width 0.4) (layer "F.Cu") (net 3))
+  (segment (start 185.8 93.39) (end 185.8 104.86) (width 0.4) (layer "F.Cu") (net 3))
   (segment (start 136.47375 93.77) (end 136.47375 95.1525) (width 0.4) (layer "F.Cu") (net 3))
+  (segment (start 140.77 109.47) (end 138.71 107.41) (width 0.4) (layer "F.Cu") (net 3))
+  (segment (start 134.74 102.03) (end 133.8675 102.9025) (width 0.4) (layer "F.Cu") (net 3))
+  (segment (start 133.8675 102.9025) (end 133.8675 104.2675) (width 0.4) (layer "F.Cu") (net 3))
   (segment (start 133.83125 94.47) (end 133.83125 95.59) (width 0.4) (layer "F.Cu") (net 3))
-  (segment (start 159.26 108.94) (end 154.89 104.57) (width 0.4) (layer "F.Cu") (net 3))
   (segment (start 138.71125 96.4925) (end 137.76875 95.55) (width 0.4) (layer "F.Cu") (net 3))
   (segment (start 182.865 88.37) (end 183.115 88.12) (width 0.4) (layer "F.Cu") (net 3))
-  (segment (start 185.8 104.86) (end 184.13 106.53) (width 0.4) (layer "F.Cu") (net 3))
-  (segment (start 134.74 102.03) (end 138.76 102.03) (width 0.4) (layer "F.Cu") (net 3))
-  (segment (start 184.365 90.91) (end 184.365 91.955) (width 0.4) (layer "F.Cu") (net 3))
   (segment (start 137.76875 95.55) (end 136.89125 95.55) (width 0.4) (layer "F.Cu") (net 3))
   (segment (start 182.865 89.14) (end 182.865 88.37) (width 0.4) (layer "F.Cu") (net 3))
-  (segment (start 138.76 102.03) (end 139.225 102.495) (width 0.4) (layer "F.Cu") (net 3))
-  (segment (start 141.3 104.57) (end 139.225 102.495) (width 0.4) (layer "F.Cu") (net 3))
-  (segment (start 184.365 91.955) (end 185.8 93.39) (width 0.4) (layer "F.Cu") (net 3))
-  (segment (start 162.94 108.94) (end 159.26 108.94) (width 0.4) (layer "F.Cu") (net 3))
-  (segment (start 139.225 102.495) (end 138.71125 101.98125) (width 0.4) (layer "F.Cu") (net 3))
+  (segment (start 184.365 90.91) (end 184.365 91.955) (width 0.4) (layer "F.Cu") (net 3))
   (segment (start 182.865 89.14) (end 182.865 89.89) (width 0.4) (layer "F.Cu") (net 3))
-  (segment (start 184.13 106.53) (end 165.35 106.53) (width 0.4) (layer "F.Cu") (net 3))
-  (segment (start 165.35 106.53) (end 162.94 108.94) (width 0.4) (layer "F.Cu") (net 3))
+  (segment (start 185.8 104.86) (end 181.19 109.47) (width 0.4) (layer "F.Cu") (net 3))
   (via (at 182.865 89.14) (size 0.8) (drill 0.4) (layers "F.Cu" "B.Cu") (net 3))
   (via (at 136.47375 93.77) (size 0.8) (drill 0.4) (layers "F.Cu" "B.Cu") (net 3))
@@
   (via (at 190.785 89.45) (size 0.8) (drill 0.4) (layers "F.Cu" "B.Cu") (net 25))
   (via (at 134.59125 87.9325) (size 0.8) (drill 0.4) (layers "F.Cu" "B.Cu") (net 25))
+  (segment (start 173.74 109.33) (end 132.67 109.33) (width 0.4) (layer "B.Cu") (net 25))
+  (segment (start 177.76 105.31) (end 173.74 109.33) (width 0.4) (layer "B.Cu") (net 25))
   (segment (start 134.6 90.87) (end 128.7875 96.6825) (width 0.4) (layer "B.Cu") (net 25))
+  (segment (start 189.625 90.61) (end 181.65 90.61) (width 0.4) (layer "B.Cu") (net 25))
+  (segment (start 177.76 94.5) (end 177.76 105.31) (width 0.4) (layer "B.Cu") (net 25))
   (segment (start 129.89 95.58) (end 128.7875 96.6825) (width 0.4) (layer "B.Cu") (net 25))
   (segment (start 128.7875 96.6825) (end 128.7875 96.96) (width 0.4) (layer "B.Cu") (net 25))
-  (segment (start 132.27 108.93) (end 128.7875 105.4475) (width 0.4) (layer "B.Cu") (net 25))
-  (segment (start 181.65 90.61) (end 177.76 94.5) (width 0.4) (layer "B.Cu") (net 25))
-  (segment (start 177.76 105.31) (end 174.14 108.93) (width 0.4) (layer "B.Cu") (net 25))
   (segment (start 134.6 87.94125) (end 134.6 90.87) (width 0.4) (layer "B.Cu") (net 25))
-  (segment (start 128.7875 105.4475) (end 128.7875 104.2675) (width 0.4) (layer "B.Cu") (net 25))
-  (segment (start 190.785 89.45) (end 189.625 90.61) (width 0.4) (layer "B.Cu") (net 25))
-  (segment (start 174.14 108.93) (end 132.27 108.93) (width 0.4) (layer "B.Cu") (net 25))
-  (segment (start 189.625 90.61) (end 181.65 90.61) (width 0.4) (layer "B.Cu") (net 25))
   (segment (start 134.59125 87.9325) (end 134.6 87.94125) (width 0.4) (layer "B.Cu") (net 25))
+  (segment (start 128.7875 105.4475) (end 128.7875 104.2675) (width 0.4) (layer "B.Cu") (net 25))
   (segment (start 128.7875 96.6825) (end 128.7875 104.2675) (width 0.4) (layer "B.Cu") (net 25))
-  (segment (start 177.76 94.5) (end 177.76 105.31) (width 0.4) (layer "B.Cu") (net 25))
+  (segment (start 190.785 89.45) (end 189.625 90.61) (width 0.4) (layer "B.Cu") (net 25))
+  (segment (start 132.67 109.33) (end 128.7875 105.4475) (width 0.4) (layer "B.Cu") (net 25))
+  (segment (start 181.65 90.61) (end 177.76 94.5) (width 0.4) (layer "B.Cu") (net 25))
   (segment (start 132.53125 95.59) (end 132.53125 98.5625) (width 0.4) (layer "F.Cu") (net 26))
   (segment (start 182.075 86.82) (end 184.245 86.82) (width 0.4) (layer "F.Cu") (net 26))
@@
   (via (at 181.645 87.25) (size 0.8) (drill 0.4) (layers "F.Cu" "B.Cu") (net 26))
   (via (at 132.53125 98.5625) (size 0.8) (drill 0.4) (layers "F.Cu" "B.Cu") (net 26))
-  (segment (start 131.3275 105.1475) (end 132.4475 106.2675) (width 0.4) (layer "B.Cu") (net 26))
   (segment (start 132.53125 98.5625) (end 131.2275 99.86625) (width 0.4) (layer "B.Cu") (net 26))
+  (segment (start 177.11 93.33) (end 181.645 88.795) (width 0.4) (layer "B.Cu") (net 26))
+  (segment (start 134.78 108.66) (end 173.4 108.66) (width 0.4) (layer "B.Cu") (net 26))
   (segment (start 131.2275 99.86625) (end 131.2275 104.1675) (width 0.4) (layer "B.Cu") (net 26))
-  (segment (start 181.645 88.795) (end 181.645 87.25) (width 0.4) (layer "B.Cu") (net 26))
+  (segment (start 173.4 108.66) (end 177.11 104.95) (width 0.4) (layer "B.Cu") (net 26))
   (segment (start 132.53125 98.5625) (end 132.57125 98.6025) (width 0.4) (layer "B.Cu") (net 26))
-  (segment (start 134.44 108.32) (end 173.74 108.32) (width 0.4) (layer "B.Cu") (net 26))
-  (segment (start 132.4475 106.2675) (end 132.4475 106.3275) (width 0.4) (layer "B.Cu") (net 26))
   (segment (start 177.11 104.95) (end 177.11 93.33) (width 0.4) (layer "B.Cu") (net 26))
+  (segment (start 132.4475 106.3275) (end 134.78 108.66) (width 0.4) (layer "B.Cu") (net 26))
+  (segment (start 132.4475 106.2675) (end 132.4475 106.3275) (width 0.4) (layer "B.Cu") (net 26))
   (segment (start 131.3275 104.2675) (end 131.3275 105.1475) (width 0.4) (layer "B.Cu") (net 26))
-  (segment (start 173.74 108.32) (end 177.11 104.95) (width 0.4) (layer "B.Cu") (net 26))
-  (segment (start 177.11 93.33) (end 181.645 88.795) (width 0.4) (layer "B.Cu") (net 26))
+  (segment (start 131.3275 105.1475) (end 132.4475 106.2675) (width 0.4) (layer "B.Cu") (net 26))
+  (segment (start 181.645 88.795) (end 181.645 87.25) (width 0.4) (layer "B.Cu") (net 26))
   (segment (start 131.2275 104.1675) (end 131.3275 104.2675) (width 0.4) (layer "B.Cu") (net 26))
-  (segment (start 132.4475 106.3275) (end 134.44 108.32) (width 0.4) (layer "B.Cu") (net 26))
   (segment (start 132.53125 98.5625) (end 132.59125 98.5625) (width 0.4) (layer "B.Cu") (net 26))
   (segment (start 197.39 81.515) (end 197.39 87.425) (width 2) (layer "F.Cu") (net 27))

Commit message: Correcting the project,cirquits and board
Parts:
- added C19: 0.1uF, Capacitor_SMD:C_1206_3216Metric, F.Cu at (125.5, 98.7)
- added C20: 0.1uF, Capacitor_SMD:C_1206_3216Metric, B.Cu at (141.6, 103.5)
- added C21: 0.1uF, Capacitor_SMD:C_1206_3216Metric, B.Cu at (141.6, 105.9)
- added R11: 2.2k, Resistor_SMD:R_1206_3216Metric, B.Cu at (141.6, 101.1)
- added R12: 2.2k, Resistor_SMD:R_1206_3216Metric, B.Cu at (141.6, 108.3)
- added SW1: SW_DIP_x02, Button_Switch_SMD:SW_DIP_SPSTx02_Slide_6.7x6.64mm_W8.61mm_P2.54mm_LowProfile, F.Cu at (131.2, 104.6)
- moved J3 18.1 mm to (154.4, 105.8)
- moved C15 3.00 mm to (139.2, 95.6)
- moved U1 0.92 mm to (132.4, 93.1)
- moved C5 0.58 mm to (128.8, 81.7)
Routing:
- net +5V: track 137.4 -> 181.0 mm
- net Net-(J3-Pin_3): track 81.4 -> 101.7 mm
- net GND: track 490.7 -> 504.0 mm
- net Net-(T1-AA): track 28.2 -> 31.1 mm
- net Net-(U1-1B2): track 15.4 -> 16.7 mm
- net Net-(U1-1B4): track 23.8 -> 22.8 mm
- net Net-(U1-1B3): track 20.1 -> 19.1 mm
- net Net-(J3-Pin_4): track 107.5 -> 106.5 mm, vias 2 -> 3
Other:
- board text added: "F1"
- board text added: "F2"
- board text removed: "K1"
- board text removed: "K2"
