File: Filter.kicad_sch (KiCad schematic)
At the start: 47 parts, among them J1 Conn_Coaxial, J3 Conn_01x04_Pin, J4 Conn_Coaxial, T1 BN-43-2402, T2 BN-43-2402, U1 SN74CBT3253, U2 SN74CBT3253

Commit message: Correcting the project,cirquits and board
Parts:
- added C19, C20, C21: 0.1uF, Capacitor_SMD:C_1206_3216Metric, symbol Device:C_Polarized
- added R11, R12: 2.2k, Resistor_SMD:R_1206_3216Metric, symbol Device:R
- added SW1: SW_DIP_x02, Button_Switch_SMD:SW_DIP_SPSTx02_Slide_6.7x6.64mm_W8.61mm_P2.54mm_LowProfile, symbol Switch:SW_DIP_x02
Connections:
- net +5V: now also C19.1, SW1.1, SW1.2
- net GND: now also C19.2, C20.2, C21.2, R11.1, R12.1
- net at J3.3 (Pin_3), U1.14 (S0), U2.14 (S0): now also C20.1, R11.2, SW1.4
- net at J3.4 (Pin_4), U1.2 (S1), U2.2 (S1): now also C21.1, R12.2, SW1.3
Other:
- moved on the sheet: J3
